File: KiCad/RelayBoardX3.kicad_sch (KiCad schematic)
At the start: 54 parts, among them J1 Conn_01x04_Male, J10 Screw_Terminal_01x02, J11 Screw_Terminal_01x02, J12 Screw_Terminal_01x02, J13 Screw_Terminal_01x02, J14 Screw_Terminal_01x02, J15 Screw_Terminal_01x02, J16 Conn_01x01_Male, J17 Conn_01x04_Male, J2 Barrel_Jack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

Commit message: Added color specs to KiCAD schema
Parts:
- D1, D2, D3: value LED -> Green
- D7: value LED -> White
- D8: value LED -> Red
- R10, R11, R12: value 330 -> 470
Changed lines of the file:
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@@
 			)
 		)
-		(property "Value" "LED"
+		(property "Value" "Green"
 			(at 187.1472 123.2408 90)
 			(effects
@@
 			)
 		)
-		(property "Value" "330"
+		(property "Value" "470"
 			(at 185.928 131.953 0)
 			(effects
@@
 			)
 		)
-		(property "Value" "LED"
+		(property "Value" "Green"
 			(at 187.1472 80.0608 90)
 			(effects
@@
 			)
 		)
-		(property "Value" "330"
+		(property "Value" "470"
 			(at 185.928 88.773 0)
 			(effects
@@
 			)
 		)
-		(property "Value" "LED"
+		(property "Value" "Green"
 			(at 187.1472 36.8808 90)
 			(effects
@@
 			)
 		)
-		(property "Value" "330"
+		(property "Value" "470"
 			(at 185.928 45.593 0)
 			(effects
@@
 			)
 		)
-		(property "Value" "LED"
+		(property "Value" "White"
 			(at 88.0872 81.3308 90)
 			(effects
@@
 			)
 		)
-		(property "Value" "LED"
+		(property "Value" "Red"
 			(at 149.0472 62.2808 90)
 			(effects
